Commit message: add simple_robot.urdf

File: robot_description/urdf/simple_robot.urdf (robot description, URDF)
Before this commit: robot robot_description, 3 links, 2 joints
Links:
- link Wheel_1: geometry collision cylinder length=0.01 radius=0.05
- link Wheel_2: geometry collision cylinder length=0.01 radius=0.05
Joints:
- joint Wheel_1: axis 0 -1 0 -> 0 1 0; origin xyz=0 -0.075 0 rpy=0 0 0 -> xyz=0 -0.07 0 rpy=0 0 0
- joint Wheel_2: axis 0 -1 0 -> 0 1 0; origin xyz=0 0.065 0 rpy=0 0 0 -> xyz=0 0.07 0 rpy=0 0 0
